File: Hardware/_autosave-MIDIborg.kicad_sch (KiCad schematic)
At the start: 42 parts

Commit message: Schematics
Connections:
- net SPI1_NSS: now also U?.77 (PA15)
- net at C?.1, Y?.1: now also U?.12 (PH0)
- net at C?.1, Y?.3: now also U?.13 (PH1)
Other:
- moved on the sheet: C?, Y?
