File: Hardware/MIDIborg.kicad_sch (KiCad schematic)
At the start: 46 parts, among them J2 8P8C, J4 8P8C, J5 Conn_ARM_JTAG_SWD_10, J6 Conn_01x11, J7 8P8C, J8 Conn_01x03, J9 Conn_01x11, P1 USB_C_Plug_USB2.0, Q1 2N7002, SW1 SW_Push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

Commit message: Finished layout
Parts:
- added C14: .1uF, Capacitor_SMD:C_0402_1005Metric_Pad0.74x0.62mm_HandSolder, symbol Device:C_Small
Connections:
- net +3V3: now also C14.2
- net GND: now also C10.1, C12.1, C13.1, C4.1, C5.1, C6.1, C7.1, C8.1, C14.1
Changed lines of the file:
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@@
   (junction (at 179.07 50.8) (diameter 0) (color 0 0 0 0)
   )
+  (junction (at 227.33 26.67) (diameter 0) (color 0 0 0 0)
+  )
   (junction (at 40.64 69.85) (diameter 0) (color 0 0 0 0)
   )
@@
   (junction (at 53.34 25.4) (diameter 0) (color 0 0 0 0)
   )
+  (junction (at 236.22 26.67) (diameter 0) (color 0 0 0 0)
+  )
   (junction (at 209.55 119.38) (diameter 0) (color 0 0 0 0)
   )
@@
   (junction (at 273.05 16.51) (diameter 0) (color 0 0 0 0)
   )
+  (junction (at 223.52 16.51) (diameter 0) (color 0 0 0 0)
+  )
   (junction (at 273.05 26.67) (diameter 0) (color 0 0 0 0)
   )
@@
     (stroke (width 0) (type default) (color 0 0 0 0))
   )
+  (wire (pts (xy 219.71 16.51) (xy 219.71 19.05))
+    (stroke (width 0) (type default) (color 0 0 0 0))
+  )
   (wire (pts (xy 177.8 45.72) (xy 179.07 45.72))
     (stroke (width 0) (type default) (color 0 0 0 0))
@@
     (stroke (width 0) (type default) (color 0 0 0 0))
   )
-  (wire (pts (xy 242.57 26.67) (xy 234.95 26.67))
+  (wire (pts (xy 219.71 26.67) (xy 219.71 24.13))
+    (stroke (width 0) (type default) (color 0 0 0 0))
+  )
+  (wire (pts (xy 242.57 26.67) (xy 236.22 26.67))
     (stroke (width 0) (type default) (color 0 0 0 0))
   )
@@
     (stroke (width 0) (type default) (color 0 0 0 0))
   )
+  (wire (pts (xy 223.52 16.51) (xy 227.33 16.51))
+    (stroke (width 0) (type default) (color 0 0 0 0))
+  )
+  (wire (pts (xy 227.33 26.67) (xy 219.71 26.67))
+    (stroke (width 0) (type default) (color 0 0 0 0))
+  )
   (wire (pts (xy 102.87 129.54) (xy 102.87 125.73))
     (stroke (width 0) (type default) (color 0 0 0 0))
@@
     (stroke (width 0) (type default) (color 0 0 0 0))
   )
+  (wire (pts (xy 236.22 26.67) (xy 236.22 29.21))
+    (stroke (width 0) (type default) (color 0 0 0 0))
+  )
   (wire (pts (xy 260.35 41.91) (xy 260.35 43.18))
     (stroke (width 0) (type default) (color 0 0 0 0))
@@
     (stroke (width 0) (type default) (color 0 0 0 0))
   )
-  (wire (pts (xy 223.52 16.51) (xy 227.33 16.51))
+  (wire (pts (xy 219.71 16.51) (xy 223.52 16.51))
     (stroke (width 0) (type default) (color 0 0 0 0))
   )
   (wire (pts (xy 53.34 25.4) (xy 64.77 25.4))
+    (stroke (width 0) (type default) (color 0 0 0 0))
+  )
+  (wire (pts (xy 236.22 26.67) (xy 234.95 26.67))
     (stroke (width 0) (type default) (color 0 0 0 0))
   )
@@
     (pin "2")
   )
+  (symbol (lib_id "power:GND") (at 236.22 29.21 0) (unit 1)
+    (in_bom yes) (on_board yes)
+    (property "Reference" "#PWR0108" (id 0) (at 236.22 35.56 0)
+      (effects (font (size 1.27 1.27)) hide)
+    )
+    (property "Value" "GND" (id 1) (at 241.3 31.75 0))
+    (property "Footprint" "" (id 2) (at 236.22 29.21 0)
+      (effects (font (size 1.27 1.27)) hide)
+    )
+    (property "Datasheet" "" (id 3) (at 236.22 29.21 0)
+      (effects (font (size 1.27 1.27)) hide)
+    )
+    (pin "1")
+  )
   (symbol (lib_id "Connector:Conn_ARM_JTAG_SWD_10") (at 130.81 38.1 0) (unit 1)
     (in_bom yes) (on_board yes)
@@
     (pin "1")
   )
+  (symbol (lib_id "Device:C_Small") (at 219.71 21.59 0) (mirror x) (unit 1)
+    (in_bom yes) (on_board yes)
+    (property "Reference" "C14" (id 0) (at 223.52 22.86 0)
+      (effects (font (size 1.27 1.27)) (justify right))
+    )
+    (property "Value" ".1uF" (id 1) (at 224.79 20.32 0)
+      (effects (font (size 1.27 1.27)) (justify right))
+    )
+    (property "Footprint" "Capacitor_SMD:C_0402_1005Metric_Pad0.74x0.62mm_HandSolder" (id 2) (at 219.71 21.59 0)
+      (effects (font (size 1.27 1.27)) hide)
+    )
+    (property "Datasheet" "~" (id 3) (at 219.71 21.59 0)
+      (effects (font (size 1.27 1.27)) hide)
+    )
+    (pin "1")
+    (pin "2")
+  )
   (symbol (lib_id "power:GND") (at 140.97 92.71 0) (unit 1)
     (in_bom yes) (on_board yes)
@@
     (in_bom yes) (on_board yes)
     (property "Reference" "R1" (id 0) (at 46.99 36.83 90))
-    (property "Value" "27" (id 1) (at 41.91 36.83 90))
+    (property "Value" "27" (id 1) (at 44.45 35.56 90))
     (property "Footprint" "Resistor_SMD:R_0402_1005Metric_Pad0.72x0.64mm_HandSolder" (id 2) (at 44.45 38.1 0)
       (effects (font (size 1.27 1.27)) hide)
@@
   (symbol (lib_id "Device:R_Small_US") (at 44.45 43.18 270) (unit 1)
     (in_bom yes) (on_board yes)
-    (property "Reference" "R2" (id 0) (at 41.91 41.91 90))
-    (property "Value" "27" (id 1) (at 46.99 41.91 90))
+    (property "Reference" "R2" (id 0) (at 46.99 41.91 90))
+    (property "Value" "27" (id 1) (at 44.45 40.64 90))
     (property "Footprint" "Resistor_SMD:R_0402_1005Metric_Pad0.72x0.64mm_HandSolder" (id 2) (at 44.45 43.18 0)
       (effects (font (size 1.27 1.27)) hide)
@@
       (reference "#PWR0107") (unit 1) (value "+3V3") (footprint "")
     )
+    (path "/589f9a50-0fdc-4b0c-819b-77bcac0e76d2"
+      (reference "#PWR0108") (unit 1) (value "GND") (footprint "")
+    )
     (path "/38285143-6cb3-43d2-8865-c620b98bd0fb"
       (reference "#PWR0110") (unit 1) (value "GND") (footprint "")
@@
       (reference "C13") (unit 1) (value ".1uF") (footprint "Capacitor_SMD:C_0402_1005Metric_Pad0.74x0.62mm_HandSolder")
     )
+    (path "/5d1ce7b1-fd56-4329-b471-73097fe9d7eb"
+      (reference "C14") (unit 1) (value ".1uF") (footprint "Capacitor_SMD:C_0402_1005Metric_Pad0.74x0.62mm_HandSolder")
+    )
     (path "/4dd1d3c3-0347-41d4-9408-3072805ea307/c28601bb-b014-43b0-978c-32717e7515c0"
